Commit message: feat: add mode name to moveit adapter to adjust the executing velocity

File: robot_description/urdf/arm380.urdf (robot description, URDF)
Before this commit: robot arm380, 8 links, 7 joints
Links:
- link Link1: mass 0.126658594854093 -> 0.3678
- link Link2: mass 0.160117926518548 -> 0.2944
- link Link3: mass 0.127031840994737 -> 0.8264
- link Link4: mass 0.0643122144006669 -> 0.2773
- link Link5: mass 0.0749072920283932 -> 0.3323
- link Link6: mass 0.0147843006339284 -> 0.0405
- link base_link: mass 0.239168935948052 -> 0.9106
Joints:
- joint joint2: axis 0 -0.999999999999993 0 -> 0 0.999999999999993 0; limit lower=-1.6232 upper=1.6232 effort=9 velocity=3.14 -> lower=-1.6572 upper=1.6572 effort=9 velocity=3.14
- joint joint3: axis 0 1 0 -> 0 -1 0; limit lower=-2.6704 upper=2.6704 effort=9 velocity=3.14 -> lower=-2.7034 upper=2.7034 effort=9 velocity=3.14
- joint joint4: limit lower=-2.7576 upper=2.7576 effort=3.3 velocity=3.14 -> lower=-2.7911 upper=2.7911 effort=3.3 velocity=3.14
- joint joint5: limit lower=-1.5359 upper=1.5359 effort=3.3 velocity=3.14 -> lower=-1.57 upper=1.57 effort=3.3 velocity=3.14

File: robot_description/urdf/arm620.urdf (robot description, URDF)
Before this commit: robot arm620, 8 links, 7 joints
Links:
- link Link1: mass 0.151006149586524 -> 1.0225
- link Link2: mass 0.343463687955357 -> 1.925
- link Link3: mass 0.13198857635385 -> 0.73
- link Link4: mass 0.0765381851810229 -> 0.5174
- link Link5: mass 0.0788266395013992 -> 0.7233
- link Link6: mass 0.0321450880318068 -> 0.0953
- link base_link: mass 0.170880634330369 -> 1.235
Joints:
- joint joint1: limit lower=-2.9670 upper=2.9670 effort=49 velocity=3.14 -> lower=-2.967 upper=2.967 effort=0 velocity=0; origin xyz=0 0 0.084 rpy=0 0 -1.5708 -> xyz=0 0 0.084 rpy=0 0 0
- joint joint2: axis 0 0 1 -> 0 0 -1; limit lower=-1.5708 upper=1.5708 effort=49 velocity=3.14 -> lower=-1.5708 upper=1.5708 effort=0 velocity=0; origin xyz=0.035 0 0.06875 rpy=1.5708 0 1.5708 -> xyz=0 0 0.068718 rpy=1.5708 0 -1.5708
- joint joint3: limit lower=-1.5708 upper=1.5708 effort=49 velocity=3.14 -> lower=-1.5708 upper=1.5708 effort=0 velocity=0; origin xyz=0 0.30025 -0.00093497 rpy=0 0 3.1416 -> xyz=0 0.30025 0 rpy=-3.1416 0 0
- joint joint4: limit lower=-2.9670 upper=2.9670 effort=9 velocity=3.14 -> lower=-2.967 upper=2.967 effort=0 velocity=0; origin xyz=0 -0.15558 -0.03403 rpy=1.5708 -1.5708 0 -> xyz=0 -0.15558 3.5E-05 rpy=1.5708 -1.5708 0
- joint joint5: axis 0 0 1 -> 1 0 0; limit lower=-1.5708 upper=1.5708 effort=9 velocity=3.14 -> lower=-1.5708 upper=1.5708 effort=0 velocity=0; origin xyz=0.034548 2.0477E-05 0.064223 rpy=9.5457E-05 1.5708 0.00060723 -> xyz=-3.5E-05 1.5362E-05 0.064223 rpy=1.5708 0 0
- joint joint6: limit lower=-2.9670 upper=2.9670 effort=9 velocity=3.14 -> lower=-2.967 upper=2.967 effort=0 velocity=0; origin xyz=-0.095552 0 -0.034587 rpy=1.5708 -1.5703 -1.5708 -> xyz=-0.00047523 0.095552 0 rpy=-1.5709 0 0
