Commit message: feat: add acceleration limits to system

File: robot_description/urdf/arm620.urdf (robot description, URDF)
Before this commit: robot arm620, 8 links, 7 joints
Joints:
- joint joint1: limit lower=-2.967 upper=2.967 effort=0 velocity=0 -> lower=-2.967 upper=2.967 effort=51 velocity=3.14
- joint joint2: limit lower=-1.5708 upper=1.5708 effort=0 velocity=0 -> lower=-1.5708 upper=1.5708 effort=51 velocity=3.14
- joint joint3: limit lower=-1.5708 upper=1.5708 effort=0 velocity=0 -> lower=-1.5708 upper=1.5708 effort=51 velocity=3.14
- joint joint4: limit lower=-2.967 upper=2.967 effort=0 velocity=0 -> lower=-2.967 upper=2.967 effort=9 velocity=3.14
- joint joint5: limit lower=-1.5708 upper=1.5708 effort=0 velocity=0 -> lower=-1.5708 upper=1.5708 effort=9 velocity=3.14
- joint joint6: limit lower=-2.967 upper=2.967 effort=0 velocity=0 -> lower=-2.967 upper=2.967 effort=9 velocity=3.14
