Commit message: refactor: Parameterize arm_type in trajectory planning strategies

File: robot_description/urdf/dual_arm620.urdf (robot description, URDF)
Before this commit: robot dual_arm620, 15 links, 14 joints
Links:
- link left_Link1: mass 0.151006149586524 -> 1.0225
- link left_Link2: mass 0.343463687955357 -> 1.925
- link left_Link3: mass 0.13198857635385 -> 0.73
- link left_Link4: mass 0.0765381851810229 -> 0.5174
- link left_Link5: mass 0.0788266395013992 -> 0.7233
- link left_Link6: mass 0.0321450880318068 -> 0.0953
- link left_base_link: mass 0.170880634330369 -> 1.235
- link right_Link1: mass 0.151006149586524 -> 1.0225
- link right_Link2: mass 0.343463687955357 -> 1.925
- link right_Link3: mass 0.13198857635385 -> 0.73
- link right_Link4: mass 0.0765381851810229 -> 0.5174
- link right_Link5: mass 0.0788266395013992 -> 0.7233
- link right_Link6: mass 0.0321450880318068 -> 0.0953
- link right_base_link: mass 0.170880634330369 -> 1.235
Joints:
- joint left_joint1: limit lower=-2.9670 upper=2.9670 effort=49 velocity=3.14 -> lower=-2.967 upper=2.967 effort=51 velocity=3.14; origin xyz=0 0 0.084 rpy=0 0 -1.5708 -> xyz=0 0 0.084 rpy=0 0 0
- joint left_joint2: axis 0 0 1 -> 0 0 -1; limit lower=-1.5708 upper=1.5708 effort=49 velocity=3.14 -> lower=-1.5708 upper=1.5708 effort=51 velocity=3.14; origin xyz=0.035 0 0.06875 rpy=1.5708 0 1.5708 -> xyz=0 0 0.068718 rpy=1.5708 0 -1.5708
- joint left_joint3: limit lower=-1.5708 upper=1.5708 effort=49 velocity=3.14 -> lower=-1.5708 upper=1.5708 effort=51 velocity=3.14; origin xyz=0 0.30025 -0.00093497 rpy=0 0 3.1416 -> xyz=0 0.30025 0 rpy=-3.1416 0 0
- joint left_joint4: limit lower=-2.9670 upper=2.9670 effort=9 velocity=3.14 -> lower=-2.967 upper=2.967 effort=9 velocity=3.14; origin xyz=0 -0.15558 -0.03403 rpy=1.5708 -1.5708 0 -> xyz=0 -0.15558 3.5E-05 rpy=1.5708 -1.5708 0
- joint left_joint5: axis 0 0 1 -> 1 0 0; origin xyz=0.034548 2.0477E-05 0.064223 rpy=9.5457E-05 1.5708 0.00060723 -> xyz=-3.5E-05 1.5362E-05 0.064223 rpy=1.5708 0 0
- joint left_joint6: limit lower=-2.9670 upper=2.9670 effort=9 velocity=3.14 -> lower=-2.967 upper=2.967 effort=9 velocity=3.14; origin xyz=-0.095552 0 -0.034587 rpy=1.5708 -1.5703 -1.5708 -> xyz=-0.00047523 0.095552 0 rpy=-1.5709 0 0
- joint right_joint1: limit lower=-2.9670 upper=2.9670 effort=49 velocity=3.14 -> lower=-2.967 upper=2.967 effort=51 velocity=3.14; origin xyz=0 0 0.084 rpy=0 0 -1.5708 -> xyz=0 0 0.084 rpy=0 0 0
- joint right_joint2: axis 0 0 1 -> 0 0 -1; limit lower=-1.5708 upper=1.5708 effort=49 velocity=3.14 -> lower=-1.5708 upper=1.5708 effort=51 velocity=3.14; origin xyz=0.035 0 0.06875 rpy=1.5708 0 1.5708 -> xyz=0 0 0.068718 rpy=1.5708 0 -1.5708
- joint right_joint3: limit lower=-1.5708 upper=1.5708 effort=49 velocity=3.14 -> lower=-1.5708 upper=1.5708 effort=51 velocity=3.14; origin xyz=0 0.30025 -0.00093497 rpy=0 0 3.1416 -> xyz=0 0.30025 0 rpy=-3.1416 0 0
- joint right_joint4: limit lower=-2.9670 upper=2.9670 effort=9 velocity=3.14 -> lower=-2.967 upper=2.967 effort=9 velocity=3.14; origin xyz=0 -0.15558 -0.03403 rpy=1.5708 -1.5708 0 -> xyz=0 -0.15558 3.5E-05 rpy=1.5708 -1.5708 0
- joint right_joint5: axis 0 0 1 -> 1 0 0; origin xyz=0.034548 2.0477E-05 0.064223 rpy=9.5457E-05 1.5708 0.00060723 -> xyz=-3.5E-05 1.5362E-05 0.064223 rpy=1.5708 0 0
- joint right_joint6: limit lower=-2.9670 upper=2.9670 effort=9 velocity=3.14 -> lower=-2.967 upper=2.967 effort=9 velocity=3.14; origin xyz=-0.095552 0 -0.034587 rpy=1.5708 -1.5703 -1.5708 -> xyz=-0.00047523 0.095552 0 rpy=-1.5709 0 0
